File: hardware/multi-channel-cremat-amplifier.kicad_sch (KiCad schematic)
At the start: 1 part

Commit message: Track 6: pcbnew board scaffold (217 footprints + nets + outline + GND zone)
hardware/gen_pcb.py builds the PCB headless from the netlist with KiCad's
pcbnew Python API: loads + places all 217 footprints, assigns every net,
draws the 225x235 mm Edge.Cuts outline + 4x M3 holes, adds an (unfilled)
GND zone, and re-applies the project net classes (pcbnew's save resets them).
Fixed J_PWR footprint name (_Horizontal) so all 217 place.

Honest scope: pcbnew has NO autorouter. The board is a net-assigned starting
point on a grid -- NOT routed and NOT a manufacturable arrangement (parts
overlap; the edge-launch MCX cutouts must move to the board edge). Signal
routing + final placement are the KiCad GUI push-and-shove router (or
FreeRouting via DSN/SES). scripts/drc.sh reports the state (499 unconnected
ratsnest + grid-placement overlaps to resolve in the GUI).

Also: scripts/drc.sh gate; status synced in development-plan + BUILD-IN-KICAD;
restored net classes (Default/power/hv_bias 1.0mm/signal) wiped by the
project rewrite.

Co-Authored-By: Claude Opus 4.8 <noreply@anthropic.com>
Parts:
- J_PWR: footprint TerminalBlock_Phoenix:TerminalBlock_Phoenix_MKDS-1,5-3_1x03_P5.00mm -> TerminalBlock_Phoenix:TerminalBlock_Phoenix_MKDS-1,5-3_1x03_P5.00mm_Horizontal
Changed lines of the file:
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@@
 			(effects (font (size 1.27 1.27)))
 		)
-		(property "Footprint" "TerminalBlock_Phoenix:TerminalBlock_Phoenix_MKDS-1,5-3_1x03_P5.00mm"
+		(property "Footprint" "TerminalBlock_Phoenix:TerminalBlock_Phoenix_MKDS-1,5-3_1x03_P5.00mm_Horizontal"
 			(at 39.37 180.34 0)
 			(hide yes)
