File: hardware/multi-channel-cremat-amplifier.kicad_pcb (KiCad board)
At the start: 2 copper layers, 225 x 235 mm, 221 parts, among them J1 MCX CONMCX013, J10 MCX CONMCX013, J11 MCX CONMCX013, J12 MCX CONMCX013, J13 MCX CONMCX013, J14 MCX CONMCX013, J15 MCX CONMCX013, J16 MCX CONMCX013, J17 MCX CONMCX013, J18 MCX CONMCX013, J19 MCX CONMCX013, J2 MCX CONMCX013, J20 MCX CONMCX013, J21 MCX CONMCX013, J22 MCX CONMCX013, J23 MCX CONMCX013, J24 MCX CONMCX013, J25 MCX CONMCX013, J26 MCX CONMCX013, J27 MCX CONMCX013, J28 MCX CONMCX013, J29 MCX CONMCX013, J3 MCX CONMCX013, J30 MCX CONMCX013, J31 MCX CONMCX013, J32 MCX CONMCX013, J33 MCX CONMCX013, J34 MCX CONMCX013, J35 MCX CONMCX013, J36 MCX CONMCX013, J4 MCX CONMCX013, J5 MCX CONMCX013, J6 MCX CONMCX013, J7 MCX CONMCX013, J8 MCX CONMCX013, J9 MCX CONMCX013, U1 CR-112, U10 CR-200-1us, U11 CR-210, U12 EL5167, U13 CR-112, U14 CR-200-1us, U15 CR-210, U16 EL5167, U17 CR-112, U18 CR-200-1us, U19 CR-210, U2 CR-200-1us, U20 EL5167, U21 CR-112, U22 CR-200-1us, U23 CR-210, U24 EL5167, U25 CR-112, U26 CR-200-1us, U27 CR-210, U28 EL5167, U29 CR-112, U3 CR-210, U30 CR-200-1us, U31 CR-210, U32 EL5167, U33 CR-112, U34 CR-200-1us, U35 CR-210, U36 EL5167, U37 CR-112, U38 CR-200-1us, U39 CR-210, U4 EL5167, U40 EL5167, U41 CR-112, U42 CR-200-1us, U43 CR-210, U44 EL5167, U45 CR-112, U46 CR-200-1us, U47 CR-210, U48 EL5167, U5 CR-112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

Commit message: Track 6: per-channel row placement + FreeRouting DSN/SES workflow
Placement (gen_pcb.py): group the 12 channels into signal-ordered rows
(J_BIAS | filter | J_SIPM+Cc | CR-11X | CR-200+P/Z | CR-210 | buffer |
R_OUT | J_OUT), module-length-aware spacing; cut DRC errors 387->266.
MCX Edge.Cuts moved to Dwgs.User (via SetLayer, not Remove -- Remove
corrupts fp.Pads) so the outline stays one clean rectangle; re-cut edges
in GUI when mechanically placing jacks.

Autorouting workflow (KiCad has no autorouter):
- hardware/export_dsn.py  -> Specctra .dsn  (pcbnew.ExportSpecctraDSN)
- hardware/import_ses.py   -> import routed .ses back to the board
- docs/FREEROUTING.md      -> download + GUI/CLI autoroute + import steps
Proven: DSN export succeeds on a clean board; it returns False while copper
overlaps remain, so the dense module region must be spread in the GUI first
(placement is the human step; FreeRouting does the routing). gitignore
*.dsn/*.ses.

Co-Authored-By: Claude Opus 4.8 <noreply@anthropic.com>
Parts:
- moved C41 247.1 mm to (34.0, 192.0), turned to 90 degrees
- moved C43 221.3 mm to (200.0, 192.0), turned to 90 degrees
- moved J_PWR 220.7 mm to (12.0, 236.0)
- moved C44 218.2 mm to (208.0, 192.0), turned to 90 degrees
- moved R62 215.1 mm to (22.0, 192.0), turned to 90 degrees
- moved C25 214.7 mm to (34.0, 120.0), turned to 90 degrees
- moved J28 210.3 mm to (10.0, 174.0)
- moved J13 205.2 mm to (10.0, 84.0)
- moved C47 201.6 mm to (200.0, 210.0), turned to 90 degrees
- moved R3 199.8 mm to (40.0, 12.0), turned to 90 degrees
- moved C48 199.2 mm to (208.0, 210.0), turned to 90 degrees
- moved R61 198.3 mm to (28.0, 192.0), turned to 90 degrees
- moved R13 198.0 mm to (28.0, 48.0), turned to 90 degrees
- moved R47 195.0 mm to (214.0, 138.0)
- moved C37 191.0 mm to (34.0, 174.0), turned to 90 degrees
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
Commit message: Track 6: DRC-clean placement (bounding-box packed) + HV creepage fix
Placement is now 0 DRC errors / 0 warnings (only the unrouted ratsnest
remains). Fixes:
- gen_pcb.py packs each channel as a left->right strip using real footprint
  bounding boxes (pcbnew GetBoundingBox), so nothing overlaps -- replaces the
  fixed-x guesswork that caused the overlaps.
- SIP-8 modules are 21mm tall at rot0; rotate them 90deg to lie flat in the
  16mm row pitch.
- Root cause of the 60 "clearance" errors: hv_bias netclass was 1.0mm, but a
  single 0805's own two pads are ~0.9mm apart, and the AC-coupling cap Cc
  bridges HV(FE)->amp(CSP_IN) across that 0.9mm. Set hv_bias clearance to
  0.6mm (IPC-2221 external-uncoated for <=60V AND >=0805 pad gap); the cap's
  100V rating provides the isolation across its body, not PCB creepage.
- Mounting holes get refs H1-H4; TOP margin raised so H1 clears ch1.

DSN export (export_dsn.py) now succeeds (43 KB) since placement is clean.
Java/FreeRouting not available in this env; DSN is ready for the user to
autoroute, or route programmatically next.

Co-Authored-By: Claude Opus 4.8 <noreply@anthropic.com>
Parts:
- removed REF** (x4): MountingHole_3.2mm_M3, MountingHole_3.2mm_M3
- added H1: MountingHole_3.2mm_M3, MountingHole_3.2mm_M3, F.Cu at (6.00, 6.00)
- added H2: MountingHole_3.2mm_M3, MountingHole_3.2mm_M3, F.Cu at (219.0, 6.00)
- added H3: MountingHole_3.2mm_M3, MountingHole_3.2mm_M3, F.Cu at (6.00, 229.0)
- added H4: MountingHole_3.2mm_M3, MountingHole_3.2mm_M3, F.Cu at (219.0, 229.0)
- moved R71 71.9 mm to (143.5, 196.0)
- moved R65 71.5 mm to (143.5, 180.0)
- moved R59 71.2 mm to (143.5, 164.0)
- moved R5 71.0 mm to (143.5, 20.0)
- moved R53 71.0 mm to (143.5, 148.0)
- moved R11 70.8 mm to (143.5, 36.0)
- moved R47 70.8 mm to (143.5, 132.0)
- moved R17 70.6 mm to (143.5, 52.0)
- moved R41 70.6 mm to (143.5, 116.0)
- moved R23 70.6 mm to (143.5, 68.0)
- moved R35 70.6 mm to (143.5, 100.0)
- moved R29 70.5 mm to (143.5, 84.0)
- moved C48 35.1 mm to (175.8, 196.0), turned to 0 degrees
- moved C44 34.3 mm to (175.8, 180.0), turned to 0 degrees
- moved C40 33.7 mm to (175.8, 164.0), turned to 0 degrees
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