File: final-board/twelve-channel/design/channel.kicad_sch (KiCad schematic)
At the start: 38 parts, among them J1 MCX edge jack 50R, J2 MCX edge jack 50R, J3 MCX edge jack 50R, J4 MCX edge jack 50R, U1 CR-112, U2 CR-200-1us, U3 CR-210, U4 THS3491

Commit message: 12ch: propagate single-channel connector fixes (Linx MCX-T + notch outline + J rot 180)
Re-tiled the 12-ch board against the updated single channel (session 8). Swapped in the user's
Linx cremat:MCX_CONMCX013-T footprint (48 instances, model rot 270 = coax off-edge); gen_pcb now
cuts 48 edge notches (24/edge) into the outline by reading each tiled MCX's Dwgs.User cutout
(instead of promoting cutouts to Edge.Cuts), waives edge_clearance for CONMCX013-T in .kicad_dru,
and rotates J_PWR/J_DAISY to 180 (funnels face out, like J5). Added MPN/Mfr/DistPN fields to the
tiled channel footprints (the regenerated single channel drops them). Deleted the old
_EdgeMount footprint + generated STEP + obsolete gen_mcx_step.py.

Verified: 48 MCX = CONMCX013-T rot(270,0,0), J49/J50 rot 180, 48 notches, ERC 0, DRC error
severity 0/0/0 (48 lib_footprint_mismatch are warning-level, intentional demotion). Render
confirms MCX lie flat off the edges. Fab regenerated.

Co-Authored-By: Claude Opus 4.8 <noreply@anthropic.com>
Parts:
- J1, J2, J3, J4: footprint cremat:MCX_CONMCX013_EdgeMount -> cremat:MCX_CONMCX013-T

Commit message: 12ch order-ready v2: socketed Cremat modules, HV-DRC fix, 1U slot-through, JLC+DigiKey ordering package
Four workstreams, all gated (ERC 0 / netlist membership identical / DRC 0 errors,
0 unconnected, 0 parity with hv_bias verified live / renders checked):

SIP-8 sockets (never solder the modules):
- All 36 module sites -> stock PinSocket_1x08 footprint (pad+courtyard identical to the
  old header placeholder). Part: Samtec SS-108-TT-2 (DK 612-SS-108-TT-2-ND) - Cremat's
  own eval-board socket; accepts the modules' 0.51x0.25mm flat pins (live-verified).
  Alt: Harwin D01-9970842. NOT Mill-Max/Preci-Dip 801 (0.7-0.9mm pins).

hv_bias 0.6mm DRC rule was silently disabled - found and fixed at the source:
- Single-channel netclass patterns 'FE'/'N_filt' lacked the leading slash and matched
  nothing -> the 07-11 reroute packed the SiPM-bias front-end at 0.2mm. Patterns now
  '*/'-prefixed; single channel re-routed with the HV rule live in the DSN; 12ch re-tiled.
- A KiCad GUI save flattened twelve-channel.kicad_pro netclasses TWICE (DRC passed
  vacuously). Pipeline now self-heals: gen_pcb re-asserts build_pro() after SaveBoard;
  fill_zones refuses to fill blind (restores netclasses + loud warning).

Enclosure: 2U -> 1U, one board per case, slot-through panels:
- Hammond RM1U1908VBK (vented; ~13W under a 40mm lid). Factory-drawing-verified:
  internal 196.85 depth x 40.09 height; socketed module stack ~32mm -> fits.
- Board W 180 -> 213.2mm: passes through a ~340x7mm milled slot in each front/rear
  panel, protruding 5mm; MCX faces ~8.6mm proud, snap-on fully in the open. Slot
  machining spec in design/SESSION_LOG.md session 14.

Ordering (ORDERING.md = master buy sheet):
- JLCPCB fab + Economic SMT assembly (live-verified incl. wizard quote: ~$74/5 boards
  HASL, large-size fee $5; Economic tier OK, edge notches OK). Package in design/fab/jlc:
  gerber zip + JLC BOM (12 lines, LCSC C-numbers, 8 Basic / 4 Extended) + CPL (246
  FIT-SMD placements). Subs documented: 10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
Parts:
- C2: Distributor PN 490-8306-1-ND -> 399-C0805C224K1RACTUCT-ND; MPN GRM21AR72A224KAC5K -> C0805C224K1RACTU; Manufacturer Murata Electronics -> KEMET
- U1, U2, U3: footprint Connector_PinHeader_2.54mm:PinHeader_1x08_P2.54mm_Vertical -> Connector_PinSocket_2.54mm:PinSocket_1x08_P2.54mm_Vertical
- U4: Distributor PN 296-49085-2-ND -> 296-49085-1-ND
Changed lines of the file:
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@@
 			(effects (font (size 1.27 1.27)))
 		)
-		(property "MPN" "GRM21AR72A224KAC5K"
+		(property "MPN" "C0805C224K1RACTU"
 			(at 93.98 115.57 0)
 			(hide yes)
 			(effects (font (size 1.27 1.27)))
 		)
-		(property "Manufacturer" "Murata Electronics"
+		(property "Manufacturer" "KEMET"
 			(at 93.98 115.57 0)
 			(hide yes)
 			(effects (font (size 1.27 1.27)))
 		)
-		(property "Distributor PN" "490-8306-1-ND"
+		(property "Distributor PN" "399-C0805C224K1RACTUCT-ND"
 			(at 93.98 115.57 0)
 			(hide yes)
@@
 			(effects (font (size 1.0 1.0)))
 		)
-		(property "Footprint" "Connector_PinHeader_2.54mm:PinHeader_1x08_P2.54mm_Vertical"
+		(property "Footprint" "Connector_PinSocket_2.54mm:PinSocket_1x08_P2.54mm_Vertical"
 			(at 120.65 120.65 0)
 			(hide yes)
@@
 			(effects (font (size 1.0 1.0)))
 		)
-		(property "Footprint" "Connector_PinHeader_2.54mm:PinHeader_1x08_P2.54mm_Vertical"
+		(property "Footprint" "Connector_PinSocket_2.54mm:PinSocket_1x08_P2.54mm_Vertical"
 			(at 185.42 120.65 0)
 			(hide yes)
@@
 			(effects (font (size 1.0 1.0)))
 		)
-		(property "Footprint" "Connector_PinHeader_2.54mm:PinHeader_1x08_P2.54mm_Vertical"
+		(property "Footprint" "Connector_PinSocket_2.54mm:PinSocket_1x08_P2.54mm_Vertical"
 			(at 250.19 120.65 0)
 			(hide yes)
@@
 			(effects (font (size 1.27 1.27)))
 		)
-		(property "Distributor PN" "296-49085-2-ND"
+		(property "Distributor PN" "296-49085-1-ND"
 			(at 317.5 115.57 0)
 			(hide yes)
